File: telluino-kicad/_autosave-telluino.kicad_sch (KiCad schematic)
At the start: 26 parts, among them J1 6P2C, U1 LE9641PQC, U2 TISP61089BDR-S

Commit message: schematics line driver done
Connections:
- net at U1.14 (VDDSW): now also U1.15 (DVDD)
- net at U1.2 (AVDD1): now also U1.35 (AVDD2)
Changed lines of the file:
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@@
   (junction (at 87.63 185.42) (diameter 0) (color 0 0 0 0)
   )
+  (junction (at 205.74 105.41) (diameter 0) (color 0 0 0 0)
+  )
   (junction (at 114.3 187.96) (diameter 0) (color 0 0 0 0)
   )
@@
     (stroke (width 0) (type default))
   )
+  (wire (pts (xy 208.28 99.06) (xy 208.28 105.41))
+    (stroke (width 0) (type default))
+  )
   (wire (pts (xy 87.63 187.96) (xy 87.63 185.42))
     (stroke (width 0) (type default))
@@
     (stroke (width 0) (type default))
   )
-  (wire (pts (xy 205.74 99.06) (xy 205.74 109.22))
+  (wire (pts (xy 205.74 99.06) (xy 205.74 105.41))
     (stroke (width 0) (type default))
   )
@@
     (stroke (width 0) (type default))
   )
+  (wire (pts (xy 208.28 105.41) (xy 205.74 105.41))
+    (stroke (width 0) (type default))
+  )
   (wire (pts (xy 165.1 153.67) (xy 176.53 153.67))
     (stroke (width 0) (type default))
@@
     (stroke (width 0) (type default))
   )
+  (wire (pts (xy 231.14 99.06) (xy 231.14 114.3))
+    (stroke (width 0) (type default))
+  )
   (wire (pts (xy 252.73 88.9) (xy 252.73 100.33))
     (stroke (width 0) (type default))
@@
     (stroke (width 0) (type default))
   )
+  (wire (pts (xy 231.14 114.3) (xy 213.36 114.3))
+    (stroke (width 0) (type default))
+  )
   (wire (pts (xy 285.75 102.87) (xy 285.75 105.41))
     (stroke (width 0) (type default))
@@
     (stroke (width 0) (type default))
   )
+  (wire (pts (xy 205.74 105.41) (xy 205.74 109.22))
+    (stroke (width 0) (type default))
+  )
   (wire (pts (xy 83.82 146.05) (xy 83.82 190.5))
     (stroke (width 0) (type default))
@@
     (stroke (width 0) (type default))
   )
-  (wire (pts (xy 213.36 99.06) (xy 213.36 113.03))
+  (wire (pts (xy 213.36 99.06) (xy 213.36 114.3))
     (stroke (width 0) (type default))
   )
@@
     )
   )
-  (netclass_flag "" (length 2.54) (shape round) (at 226.06 109.22 180) (fields_autoplaced)
+  (netclass_flag "" (length 2.54) (shape round) (at 226.06 109.22 180)
     (effects (font (size 1.27 1.27)) (justify right bottom))
-    (property "Netclass" "VDHP1" (at 226.7585 111.76 0)
+    (property "Netclass" "VDHP1" (at 227.33 110.49 90)
       (effects (font (size 1.27 1.27) italic) (justify left))
     )
@@
   (netclass_flag "" (length 2.54) (shape round) (at 205.74 107.95 180)
     (effects (font (size 1.27 1.27)) (justify right bottom))
-    (property "Netclass" "3.3VA1" (at 203.2 113.03 0)
+    (property "Netclass" "3.3VA" (at 203.2 113.03 0)
       (effects (font (size 1.27 1.27) italic) (justify left))
     )
@@
     )
   )
-  (netclass_flag "" (length 2.54) (shape round) (at 213.36 113.03 180)
+  (netclass_flag "" (length 2.54) (shape round) (at 213.36 114.3 180)
     (effects (font (size 1.27 1.27)) (justify right bottom))
-    (property "Netclass" "3.3V" (at 213.36 118.11 0)
+    (property "Netclass" "3.3V" (at 213.36 119.38 0)
       (effects (font (size 1.27 1.27) italic) (justify left))
     )
@@
     )
   )
-  (symbol (lib_id "LE9641:LE9641PQC") (at 167.64 99.06 90) (unit 2)
+  (symbol (lib_name "LE9641PQC_1") (lib_id "LE9641:LE9641PQC") (at 167.64 99.06 90) (unit 2)
     (in_bom yes) (on_board yes) (dnp no) (fields_autoplaced)
     (property "Reference" "U1" (at 203.2 62.23 90)
@@
   (symbol (lib_id "LE9641:LE9641PQC") (at 203.2 125.73 0) (unit 1)
     (in_bom yes) (on_board yes) (dnp no) (fields_autoplaced)
-    (property "Reference" "U1" (at 233.68 116.84 0)
+    (property "Reference" "U1" (at 240.03 161.29 90)
       (effects (font (size 1.524 1.524)))
     )
-    (property "Value" "LE9641PQC" (at 233.68 119.38 0)
+    (property "Value" "LE9641PQC" (at 237.49 161.29 90)
       (effects (font (size 1.524 1.524)))
     )
