File: telluino-kicad/arduino_controllers.kicad_sch (KiCad schematic)
At the start: 1 part

Commit message: schematic done
Parts:
- removed A1: Arduino_UNO_R3, Module:Arduino_UNO_R3, symbol MCU_Module:Arduino_UNO_R3
- added C12, C13: 0.1uF, symbol Device:C_Small
- added C14, C18, C19, C20: 1uF, symbol Device:C_Small
- added C15, C21: 4.7uF_16V, symbol Device:C_Polarized_Small
- added C16, C17: 100nF, symbol Device:C_Small
- added D1: PWR Green, symbol Device:LED
- added D2: Red Rx, symbol Device:LED
- added D3: Green Tx, symbol Device:LED
- added D4: RUN Blue, symbol Device:LED
- added F1: MF-MSMF050-2, my_lib:FUSM4632X85, symbol MSMF050:MF-MSMF050-2
- added J2: USB_A, Connector_USB:USB_A_CNCTech_1001-011-01101_Horizontal, symbol Connector:USB_A
- added RN1, RN2: 4*1K, my_lib:SOIC127P780X210-8N, symbol Device:R_Pack04
- added SW1: SW_Push, symbol Switch:SW_Push
- added U3: DS2433S+, my_lib:SOIC127P780X210-8N, symbol my_lib:DS2433S+
- added U4: ATmega328P-A, Package_QFP:TQFP-32_7x7mm_P0.8mm, symbol MCU_Microchip_ATmega:ATmega328P-A
- added U5: CH340G, Package_SO:SOIC-16_3.9x9.9mm_P1.27mm, symbol Interface_USB:CH340G
- added U6: SS1P3L, my_lib:DO220AAL, symbol SS1P3L:SS1P3L
- added U7: LM1117DT-5.0, Package_TO_SOT_SMD:TO-252-3_TabPin2, symbol Regulator_Linear:LM1117DT-5.0
- added Y1: 16MHz, Crystal:Crystal_HC49-U-3Pin_Vertical, symbol Device:Crystal_GND2
- added Y2: 12MHz, Crystal:Crystal_HC49-U-3Pin_Vertical, symbol Device:Crystal_GND2
Connections:
- new net: C13.2, RN1.6 (R3.2), SW1.1, U4.29 (~{RESET}/PC6)
- new net: C17.2, U4.20 (AREF)
- new net: D2.1 (K), RN1.8 (R1.2), U5.2 (TXD)
- new net: D2.2 (A), RN2.1 (R1.1)
- new net: C13.1, U5.13 (~{DTR})
- new net: D1.2 (A), RN1.5 (R4.2)
- new net: U4.8 (XTAL2/PB7), Y1.1
- new net: U4.7 (XTAL1/PB6), Y1.3
- new net: U5.7 (XI), Y2.1
- new net: U5.8 (XO), Y2.3
- new net: RN1.1 (R1.1), U4.30 (PD0(RX0))
- new net: RN1.2 (R2.1), U4.31 (PD1(TX0))
- new net: D3.1 (K), RN1.7 (R2.2), U5.3 (RXD)
- new net: D3.2 (A), RN2.2 (R2.1)
- new net: F1.1, J2.1 (VBUS)
- new net: J2.2 (D-), U5.6 (UD-)
- new net: J2.3 (D+), U5.5 (UD+)
- new net: D4.2 (A), RN2.6 (R3.2)
- new net +3.3V: C12.2, U5.4 (V3)
- new net +5V: C14.1, C18.2, C19.2, C20.2, C21.1, RN1.3 (R3.1), RN1.4 (R4.1), RN2.5 (R4.2), RN2.7 (R2.2), RN2.8 (R1.2), U4.18 (AVCC), U4.4 (VCC), U4.6 (VCC), U5.16 (VCC), U6.P$1 (K), U7.2 (VO)
- new net 1WIRE: RN2.4 (R4.1), U3.3 (DATA), U4.12 (PB0)
- new net ADC6: U4.19 (ADC6)
- new net ADC7: U4.22 (ADC7)
- new net CS_N_5: U4.14 (PB2(*SS))
- new net DCLK_5: U4.17 (PB5(SCK))
- new net DIN_5: U4.15 (PB3(MOSI))
- new net DOUT_5: U4.16 (PB4(MISO))
- new net DRA_5: U4.27 (PC4(SDA))
- new net DXA_5: U4.26 (PC3)
- new net FS_5: U4.25 (PC2)
- new net GNDD: C12.1, C14.2, C15.2, C16.1, C17.1, C18.1, C19.1, C20.1, C21.2, D1.1 (K), D4.1 (K), J2.4 (GND), J2.5 (Shield), SW1.2, U3.4 (GND), U4.21 (GND), U4.3 (GND), U4.5 (GND), U5.1 (GND), U7.1 (GND), Y1.2, Y2.2
- new net INT_N: U4.32 (PD2(INT0))
- new net PC0: U4.23 (PC0)
- new net PC1: U4.24 (PC1)
- new net PCLK_5: U4.28 (PC5(SCL))
- new net PD2: U4.1 (PD3(INT1))
- new net PD4: U4.2 (PD4)
- new net PD5: U4.9 (PD5)
- new net PD6: U4.10 (PD6)
- new net PD7: U4.11 (PD7)
- new net RUN: RN2.3 (R3.1), U4.13 (PB1)
- new net VBUS: C15.1, C16.2, F1.2, U6.P$2 (A)
- new net VCC: U7.3 (VI)
Other:
- note added: "* Place near pin 4, 6, 18"

Commit message: ready_placement
Parts:
- removed C14: 1uF, symbol Device:C_Small
- removed J2: USB_A, Connector_USB:USB_A_CNCTech_1001-011-01101_Horizontal, symbol Connector:USB_A
- removed U3: DS2433S+, my_lib:SOIC127P780X210-8N, symbol my_lib:DS2433S+
- removed U5: CH340G, Package_SO:SOIC-16_3.9x9.9mm_P1.27mm, symbol Interface_USB:CH340G
- removed U7: LM1117DT-5.0, Package_TO_SOT_SMD:TO-252-3_TabPin2, symbol Regulator_Linear:LM1117DT-5.0
- removed Y2: 12MHz, Crystal:Crystal_HC49-U-3Pin_Vertical, symbol Device:Crystal_GND2
- added C22: 100nF, Capacitor_SMD:C_0603_1608Metric, symbol Device:C_Small
- added C23: 10uF_16V, Capacitor_THT:CP_Radial_D5.0mm_P2.50mm, symbol Device:C_Polarized_Small
- added C25, C26: 0.1uF, Capacitor_SMD:C_0603_1608Metric, symbol Device:C_Small
- added D5: RUN Blue, LED_SMD:LED_0603_1608Metric, symbol Device:LED
- added D6: Green Tx, LED_SMD:LED_0603_1608Metric, symbol Device:LED
- added D7: OP Orange, LED_SMD:LED_0603_1608Metric, symbol Device:LED
- added F2: MF-MSMF050-2, my_lib:FUSM4632X85, symbol MSMF050:MF-MSMF050-2
- added J3: USB_B, Connector_USB:USB_B_Lumberg_2411_02_Horizontal, symbol Connector:USB_B
- added J4: USB_A, Connector_USB:USB_A_CNCTech_1001-011-01101_Horizontal, symbol Connector:USB_A
- added U10, U3, U7: SS1P3L, my_lib:DO220AAL, symbol SS1P3L:SS1P3L
- added U5, U9: CH340C, Package_SO:SOIC-16_3.9x9.9mm_P1.27mm, symbol Interface_USB:CH340C
- C12, C13, C16, C17, C18, C19, C20: footprint (none) -> Capacitor_SMD:C_0603_1608Metric
- C15, C21: value 4.7uF_16V -> 10uF_16V; footprint (none) -> Capacitor_THT:CP_Radial_D5.0mm_P2.50mm
- D1, D2, D3: footprint (none) -> LED_SMD:LED_0603_1608Metric
- D4: value RUN Blue -> Red Rx; footprint (none) -> LED_SMD:LED_0603_1608Metric
- SW1: footprint (none) -> Button_Switch_SMD:SW_SPST_TL3305A
Connections:
- net +3.3V: now also U10.P$1 (K), U7.P$1 (K); no longer C12.2
- net +5V: now also RN2.6 (R3.2), U3.P$1 (K), U5.16 (VCC), U9.16 (VCC)
- net GNDD: now also C22.1, C23.2, C26.1, D5.1 (K), D7.1 (K), J3.4 (GND), J3.5 (Shield), J4.4 (GND), J4.5 (Shield), U5.1 (GND), U9.1 (GND); no longer D4.1 (K)
- net PD4: now also D4.1 (K), U9.3 (RXD)
- net PD5: now also D6.1 (K), U9.2 (TXD)
- net RUN: now also RN1.2 (R2.1); no longer RN2.3 (R3.1)
- net RESET*: now reaches C13.2, RN1.6 (R3.2), SW1.1, U4.29 (~{RESET}/PC6)
- net RESET*: now also C25.2
- net at D2.1 (K): now also U4.30 (PD0(RX0)), U5.2 (TXD); no longer RN1.8 (R1.2)
- net at C13.1: now also U5.13 (~{DTR})
- net PB0: now reaches RN1.1 (R1.1)
- net PB0: now also U4.12 (PB0); no longer U4.30 (PD0(RX0))
- net at U4.31 (PD1(TX0)): now also D3.1 (K), U5.3 (RXD); no longer RN1.2 (R2.1)
- net at RN1.7 (R2.2): now also D5.2 (A); no longer D3.1 (K)
- net at F1.1: now also J3.1 (VBUS)
- net at D4.2 (A): now also RN2.4 (R4.1); no longer RN2.6 (R3.2)
- removed net 1WIRE: RN2.4 (R4.1), U4.12 (PB0)
- net VBUS renamed +5VL
- new net: J3.2 (D-), U5.6 (UD-)
- new net: J3.3 (D+), U5.5 (UD+)
- new net: D6.2 (A), RN2.3 (R3.1)
- new net: C25.1, U9.13 (~{DTR})
- new net: F2.1, J4.1 (VBUS)
- new net: J4.2 (D-), U9.6 (UD-)
- new net: J4.3 (D+), U9.5 (UD+)
- new net: D7.2 (A), RN1.8 (R1.2)
- new net +3.3VA: C12.2, U5.4 (V3), U7.P$2 (A)
- new net +3.3VP: C26.2, U10.P$2 (A), U9.4 (V3)
- new net +5VP: C22.2, C23.1, F2.2, U3.P$2 (A)
Other:
- moved on the sheet: C13, C15, C16, D1, D2, D3, F1, RN1, RN2, U6

Commit message: half placed
Parts:
- renumbered D5 to D2, D7 to D3, D2 to D4, D3 to D5, D4 to D6, D6 to D7
