File: telluino-kicad/buck_boot_supply.kicad_sch (KiCad schematic)
At the start: 22 parts, among them Q1 ZXTP2012Z, Q3 MMBT3904

Commit message: schematic done
Connections:
- net GNDA: no longer CCS1.2, CFL1.1, CFL2.2, CPF1.1, CPF2.2, RLM1.2, RLM2.2, RLM3.2, RLM4.2, RTH1.2
- net SWISY1 renamed SWISY
- net SWOUTY1 renamed SWOUTY
- net VBAT1 renamed VBAT
- net VBSENSE1 renamed VBSENSE
- new net GNDD: CCS1.2, CFL1.1, CFL2.2, CPF1.1, CPF2.2, RLM1.2, RLM2.2, RLM3.2, RLM4.2, RTH1.2

Commit message: ready_placement
Parts:
- CCS1, CSW1: footprint Capacitor_SMD:C_0805_2012Metric -> Capacitor_SMD:C_0603_1608Metric
- CFL1: footprint Capacitor_THT:CP_Radial_D10.0mm_P2.50mm -> Capacitor_THT:CP_Radial_D8.0mm_P3.50mm
- CFL2: footprint Capacitor_SMD:C_0201_0603Metric -> Capacitor_SMD:C_0603_1608Metric
- CPF1: footprint Capacitor_THT:CP_Radial_D10.0mm_P2.50mm -> Capacitor_THT:CP_Radial_D12.5mm_P5.00mm
- CPF2: footprint Capacitor_SMD:C_0603_1608Metric -> Capacitor_SMD:C_0603_1608Metric_Pad1.08x0.95mm_HandSolder
- CS1: footprint Capacitor_SMD:C_0402_1005Metric -> Capacitor_SMD:C_0603_1608Metric
- DSW1: footprint SMA_DIO -> Diode_SMD:D_SMA
- RB1, RP1: footprint Resistor_SMD:R_01005_0402Metric -> Resistor_SMD:R_0603_1608Metric
- RCS1: footprint Resistor_SMD:R_0603_1608Metric -> Resistor_SMD:R_0402_1005Metric
- RLM1, RLM2, RLM3, RLM4, RTH1: footprint Resistor_SMD:R_01005_0402Metric -> Resistor_SMD:R_0402_1005Metric
Changed lines of the file:
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@@
       (effects (font (size 1.27 1.27)) (justify left))
     )
-    (property "Footprint" "Resistor_SMD:R_01005_0402Metric" (at 104.902 66.04 90)
+    (property "Footprint" "Resistor_SMD:R_0603_1608Metric" (at 104.902 66.04 90)
       (effects (font (size 1.27 1.27)) hide)
     )
@@
       (effects (font (size 1.27 1.27)) (justify left))
     )
-    (property "Footprint" "Capacitor_SMD:C_0201_0603Metric" (at 162.56 85.09 0)
+    (property "Footprint" "Capacitor_SMD:C_0603_1608Metric" (at 162.56 85.09 0)
       (effects (font (size 1.27 1.27)) hide)
     )
@@
       (effects (font (size 1.27 1.27)) (justify left))
     )
-    (property "Footprint" "Resistor_SMD:R_01005_0402Metric" (at 183.642 115.57 90)
+    (property "Footprint" "Resistor_SMD:R_0402_1005Metric" (at 183.642 115.57 90)
       (effects (font (size 1.27 1.27)) hide)
     )
@@
       (effects (font (size 1.27 1.27)))
     )
-    (property "Footprint" "Resistor_SMD:R_0603_1608Metric" (at 171.45 110.998 90)
+    (property "Footprint" "Resistor_SMD:R_0402_1005Metric" (at 171.45 110.998 90)
       (effects (font (size 1.27 1.27)) hide)
     )
@@
       (effects (font (size 1.27 1.27)) (justify left))
     )
-    (property "Footprint" "Resistor_SMD:R_01005_0402Metric" (at 139.192 115.57 90)
+    (property "Footprint" "Resistor_SMD:R_0402_1005Metric" (at 139.192 115.57 90)
       (effects (font (size 1.27 1.27)) hide)
     )
@@
       (effects (font (size 1.27 1.27)) (justify left))
     )
-    (property "Footprint" "Capacitor_SMD:C_0603_1608Metric" (at 195.58 85.09 0)
+    (property "Footprint" "Capacitor_SMD:C_0603_1608Metric_Pad1.08x0.95mm_HandSolder" (at 195.58 85.09 0)
       (effects (font (size 1.27 1.27)) hide)
     )
@@
       (effects (font (size 1.27 1.27)) (justify left))
     )
-    (property "Footprint" "Resistor_SMD:R_01005_0402Metric" (at 149.352 115.57 90)
+    (property "Footprint" "Resistor_SMD:R_0402_1005Metric" (at 149.352 115.57 90)
       (effects (font (size 1.27 1.27)) hide)
     )
@@
       (effects (font (size 1.27 1.27)) (justify left))
     )
-    (property "Footprint" "Capacitor_THT:CP_Radial_D10.0mm_P2.50mm" (at 207.01 85.09 0)
+    (property "Footprint" "Capacitor_THT:CP_Radial_D12.5mm_P5.00mm" (at 207.01 85.09 0)
       (effects (font (size 1.27 1.27)) hide)
     )
@@
       (effects (font (size 1.27 1.27)) (justify left))
     )
-    (property "Footprint" "Capacitor_SMD:C_0805_2012Metric" (at 93.98 63.5 0)
+    (property "Footprint" "Capacitor_SMD:C_0603_1608Metric" (at 93.98 63.5 0)
       (effects (font (size 1.27 1.27)) hide)
     )
@@
       (effects (font (size 1.27 1.27)) (justify left))
     )
-    (property "Footprint" "Capacitor_SMD:C_0805_2012Metric" (at 176.53 115.57 0)
+    (property "Footprint" "Capacitor_SMD:C_0603_1608Metric" (at 176.53 115.57 0)
       (effects (font (size 1.27 1.27)) hide)
     )
@@
       (effects (font (size 1.27 1.27)) (justify left))
     )
-    (property "Footprint" "Resistor_SMD:R_01005_0402Metric" (at 159.512 115.57 90)
+    (property "Footprint" "Resistor_SMD:R_0402_1005Metric" (at 159.512 115.57 90)
       (effects (font (size 1.27 1.27)) hide)
     )
@@
       (effects (font (size 1.524 1.524)))
     )
-    (property "Footprint" "SMA_DIO" (at 152.4 77.47 0)
+    (property "Footprint" "Diode_SMD:D_SMA" (at 152.4 77.47 0)
       (effects (font (size 1.27 1.27) italic) hide)
     )
@@
       (effects (font (size 1.27 1.27)) (justify left))
     )
-    (property "Footprint" "Capacitor_SMD:C_0402_1005Metric" (at 93.98 80.01 0)
+    (property "Footprint" "Capacitor_SMD:C_0603_1608Metric" (at 93.98 80.01 0)
       (effects (font (size 1.27 1.27)) hide)
     )
@@
       (effects (font (size 1.27 1.27)) (justify left))
     )
-    (property "Footprint" "Resistor_SMD:R_01005_0402Metric" (at 129.032 115.57 90)
+    (property "Footprint" "Resistor_SMD:R_0402_1005Metric" (at 129.032 115.57 90)
       (effects (font (size 1.27 1.27)) hide)
     )
@@
       (effects (font (size 1.27 1.27)) (justify left))
     )
-    (property "Footprint" "Resistor_SMD:R_01005_0402Metric" (at 84.582 82.55 90)
+    (property "Footprint" "Resistor_SMD:R_0603_1608Metric" (at 84.582 82.55 90)
       (effects (font (size 1.27 1.27)) hide)
     )
@@
       (effects (font (size 1.27 1.27)) (justify left))
     )
-    (property "Footprint" "Capacitor_THT:CP_Radial_D10.0mm_P2.50mm" (at 175.26 85.09 0)
-      (effects (font (size 1.27 1.27)) hide)
-    )
+    (property "Footprint" "Capacitor_THT:CP_Radial_D8.0mm_P3.50mm" (at 175.26 85.09 0)
+      (effects (font (size 1.27 1.27)) hide)
+    )

Commit message: half placed
Parts:
- added CSWB1: 220uF/25V, Capacitor_THT:CP_Radial_D10.0mm_P5.00mm, symbol Device:C_Polarized_US
- CPF1: value 47uF/100V -> 1uF/100V; footprint Capacitor_THT:CP_Radial_D12.5mm_P5.00mm -> Capacitor_THT:CP_Radial_D8.0mm_P3.50mm
Connections:
- net GNDA: now also CSWB1.2
- net VSW renamed +5V
- net +5V: now also CSWB1.1
Changed lines of the file:
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@@
   (junction (at 140.97 123.19) (diameter 0) (color 0 0 0 0)
   )
-  (junction (at 130.81 57.15) (diameter 0) (color 0 0 0 0)
+  (junction (at 97.79 143.51) (diameter 0) (color 0 0 0 0)
   )
   (junction (at 176.53 109.22) (diameter 0) (color 0 0 0 0)
@@
     (stroke (width 0) (type default))
   )
+  (wire (pts (xy 97.79 143.51) (xy 97.79 144.78))
+    (stroke (width 0) (type default))
+  )
   (wire (pts (xy 140.97 111.76) (xy 140.97 109.22))
     (stroke (width 0) (type default))
@@
     (stroke (width 0) (type default))
   )
-  (wire (pts (xy 130.81 55.88) (xy 130.81 57.15))
-    (stroke (width 0) (type default))
-  )
   (wire (pts (xy 195.58 92.71) (xy 207.01 92.71))
     (stroke (width 0) (type default))
@@
     (stroke (width 0) (type default))
   )
+  (wire (pts (xy 97.79 156.21) (xy 97.79 152.4))
+    (stroke (width 0) (type default))
+  )
   (wire (pts (xy 175.26 92.71) (xy 175.26 96.52))
     (stroke (width 0) (type default))
@@
     (stroke (width 0) (type default))
   )
-  (wire (pts (xy 130.81 57.15) (xy 130.81 59.69))
-    (stroke (width 0) (type default))
-  )
   (wire (pts (xy 93.98 71.12) (xy 106.68 71.12))
     (stroke (width 0) (type default))
@@
     (stroke (width 0) (type default))
   )
+  (wire (pts (xy 97.79 143.51) (xy 90.17 143.51))
+    (stroke (width 0) (type default))
+  )
   (wire (pts (xy 106.68 59.69) (xy 106.68 62.23))
     (stroke (width 0) (type default))
@@
     (stroke (width 0) (type default))
   )
+  (wire (pts (xy 97.79 143.51) (xy 106.68 143.51))
+    (stroke (width 0) (type default))
+  )
   (wire (pts (xy 114.3 86.36) (xy 120.65 86.36))
     (stroke (width 0) (type default))
   )
-  (wire (pts (xy 130.81 57.15) (xy 142.24 57.15))
+  (wire (pts (xy 130.81 59.69) (xy 142.24 59.69))
     (stroke (width 0) (type default))
   )
@@
     )
   )
-  (global_label "VSW" (shape input) (at 142.24 57.15 0) (fields_autoplaced)
+  (global_label "VSW" (shape input) (at 142.24 59.69 0) (fields_autoplaced)
     (effects (font (size 1.27 1.27)) (justify left))
-    (property "Intersheetrefs" "${INTERSHEET_REFS}" (at 148.8953 57.15 0)
+    (property "Intersheetrefs" "${INTERSHEET_REFS}" (at 148.8953 59.69 0)
       (effects (font (size 1.27 1.27)) (justify left) hide)
+    )
+  )
+  (global_label "+5V" (shape passive) (at 90.17 143.51 180) (fields_autoplaced)
+    (effects (font (size 1.27 1.27)) (justify right))
+    (property "Intersheetrefs" "${INTERSHEET_REFS}" (at 84.505 143.51 0)
+      (effects (font (size 1.27 1.27)) (justify right) hide)
     )
   )
@@
     )
   )
+  (global_label "VSW" (shape passive) (at 106.68 143.51 0) (fields_autoplaced)
+    (effects (font (size 1.27 1.27)) (justify left))
+    (property "Intersheetrefs" "${INTERSHEET_REFS}" (at 112.224 143.51 0)
+      (effects (font (size 1.27 1.27)) (justify left) hide)
+    )
+  )
   (global_label "SWISY" (shape output) (at 195.58 109.22 0) (fields_autoplaced)
     (effects (font (size 1.27 1.27)) (justify left))
@@
     )
   )
-  (netclass_flag "" (length 2.54) (shape round) (at 130.81 55.88 0) (fields_autoplaced)
-    (effects (font (size 1.27 1.27)) (justify left bottom))
-    (property "Netclass" "VSW" (at 131.5085 53.34 0)
-      (effects (font (size 1.27 1.27) italic) (justify left))
-    )
-  )
   (netclass_flag "" (length 2.54) (shape round) (at 120.65 82.55 0) (fields_autoplaced)
     (effects (font (size 1.27 1.27)) (justify left bottom))
@@
     )
   )
+  (symbol (lib_id "power:GNDA") (at 97.79 156.21 0) (unit 1)
+    (in_bom yes) (on_board yes) (dnp no) (fields_autoplaced)
+    (property "Reference" "#PWR013" (at 97.79 162.56 0)
+      (effects (font (size 1.27 1.27)) hide)
+    )
+    (property "Value" "GNDA" (at 97.79 161.29 0)
+      (effects (font (size 1.27 1.27)))
+    )
+    (property "Footprint" "" (at 97.79 156.21 0)
+      (effects (font (size 1.27 1.27)) hide)
+    )
+    (property "Datasheet" "" (at 97.79 156.21 0)
+      (effects (font (size 1.27 1.27)) hide)
+    )
+    (pin "1")
+    (instances
+      (project "telluino"
+        (path "/3bd12265-4173-4d6b-91eb-5b474bc7bb16"
+          (reference "#PWR013") (unit 1)
+        )
+        (path "/3bd12265-4173-4d6b-91eb-5b474bc7bb16/de427dad-d24a-4626-86e4-06027dc022b9"
+          (reference "#PWR010") (unit 1)
+        )
+        (path "/3bd12265-4173-4d6b-91eb-5b474bc7bb16/14dbbff9-3cfb-49d8-8c76-2abe81712cc0"
+          (reference "#PWR021") (unit 1)
+        )
+        (path "/3bd12265-4173-4d6b-91eb-5b474bc7bb16/47fd81fb-bb6e-4c28-8162-8bf84b70df9e"
+          (reference "#PWR010") (unit 1)
+        )
+      )
+    )
+  )
   (symbol (lib_id "Device:R") (at 151.13 115.57 0) (unit 1)
     (in_bom yes) (on_board yes) (dnp no)
@@
       (effects (font (size 1.27 1.27)) (justify left))
     )
-    (property "Value" "47uF/100V" (at 210.82 83.82 90)
-      (effects (font (size 1.27 1.27)) (justify left))
-    )
-    (property "Footprint" "Capacitor_THT:CP_Radial_D12.5mm_P5.00mm" (at 207.01 85.09 0)
+    (property "Value" "1uF/100V" (at 210.82 83.82 90)
+      (effects (font (size 1.27 1.27)) (justify left))
+    )
+    (property "Footprint" "Capacitor_THT:CP_Radial_D8.0mm_P3.50mm" (at 207.01 85.09 0)
       (effects (font (size 1.27 1.27)) hide)
     )
@@
         )
       )
+    )
+  )
+  (symbol (lib_id "Device:C_Polarized_US") (at 97.79 148.59 0) (unit 1)
+    (in_bom yes) (on_board yes) (dnp no)
+    (property "Reference" "CSWB1" (at 90.17 152.4 0)
+      (effects (font (size 1.27 1.27)) (justify left))
+    )
+    (property "Value" "220uF/25V" (at 99.06 152.4 0)
+      (effects (font (size 1.27 1.27)) (justify left))
+    )
+    (property "Footprint" "Capacitor_THT:CP_Radial_D10.0mm_P5.00mm" (at 97.79 148.59 0)
+      (effects (font (size 1.27 1.27)) hide)
+    )
+    (property "Datasheet" "~" (at 97.79 148.59 0)
+      (effects (font (size 1.27 1.27)) hide)
+    )
+    (pin "1")
+    (pin "2")
+    (instances
+      (project "telluino"
+        (path "/3bd12265-4173-4d6b-91eb-5b474bc7bb16"
+          (reference "CSWB1") (unit 1)
+        )
+        (path "/3bd12265-4173-4d6b-91eb-5b474bc7bb16/de427dad-d24a-4626-86e4-06027dc022b9"
+          (reference "CSWB1") (unit 1)
+        )
+        (path "/3bd12265-4173-4d6b-91eb-5b474bc7bb16/14dbbff9-3cfb-49d8-8c76-2abe81712cc0"
+          (reference "CSWB1") (unit 1)
+        )
+        (path "/3bd12265-4173-4d6b-91eb-5b474bc7bb16/47fd81fb-bb6e-4c28-8162-8bf84b70df9e"
+          (reference "CSWB1") (unit 1)
+        )
+      )
