File: telluino-kicad/slic.kicad_sch (KiCad schematic)
At the start: 26 parts, among them J1 6P2C, U1 LE9641PQC, U2 TISP61089BDR-S

Commit message: schematic done
Parts:
- removed F1: Polyfuse, Resistor_SMD:R_0201_0603Metric, symbol Device:Polyfuse
- removed F2: Polyfuse, symbol Device:Polyfuse
- added CSWB1: 220uF/25V, Capacitor_THT:CP_Radial_D10.0mm_P2.50mm, symbol Device:C_Polarized_US
- added CV1: 4.7uF/8.3V, Capacitor_SMD:C_0201_0603Metric_Pad0.64x0.40mm_HandSolder, symbol Device:C_Small
- added CV2: 1uF/8.3V, Capacitor_SMD:C_0201_0603Metric_Pad0.64x0.40mm_HandSolder, symbol Device:C_Small
- added CVA1: 0.1uF/16V, Capacitor_SMD:C_0201_0603Metric_Pad0.64x0.40mm_HandSolder, symbol Device:C_Small
- added CVD1: 0.01uF/16V, Capacitor_SMD:C_0201_0603Metric_Pad0.64x0.40mm_HandSolder, symbol Device:C_Small
- added CVID1: 0.1uF/18V, Capacitor_SMD:C_0201_0603Metric_Pad0.64x0.40mm_HandSolder, symbol Device:C_Small
- added JP1: A_D_Ground_Bridge, symbol Jumper:SolderJumper_2_Bridged
- added PTC1: ~, symbol my_lib:MF-SD013/250
- added RV1: 2R0 5%, Resistor_THT:R_Axial_DIN0309_L9.0mm_D3.2mm_P12.70mm_Horizontal, symbol Device:R_Small
Connections:
- net VDHPI is gone; now on net +3.3V: U1.23 (VDDHPI)
- net +3.3V: now also CSWB1.1, CV1.2, CVD1.2, CVID1.2, RV1.1
- net 3.3VA: now also CV2.2, CVA1.2, RV1.2
- net GNDA: now also CSWB1.2, CV1.1, CV2.1, CVA1.1, CVD1.1, CVID1.1, JP1.1 (A)
- net VBAT1: no longer C4.2, U1.48 (VBAT1)
- net CS0_N renamed CS_N
- net INT0_N renamed INT_N
- net SWISY1 renamed SWISY
- net SWOUTY1 renamed SWOUTY
- net VBSENSE1 renamed VBSENSE
- new net GNDD: JP1.2 (B)
- new net VBAT: C4.2, U1.48 (VBAT1)
Other:
- note added: "Locate CVDx near DVDD and CVAx near AVDD pins."

Commit message: ready_placement
Parts:
- C1, C10, C11, C4, C6, C7, C8, C9, CV1, CV2, CVA1, CVD1, CVID1: footprint Capacitor_SMD:C_0201_0603Metric_Pad0.64x0.40mm_HandSolder -> Capacitor_SMD:C_0603_1608Metric
- C2: footprint Capacitor_SMD:C_0603_1608Metric_Pad1.08x0.95mm_HandSolder -> Capacitor_SMD:C_0603_1608Metric
- C3: footprint (none) -> Capacitor_SMD:C_0603_1608Metric
- CSWB1: footprint Capacitor_THT:CP_Radial_D10.0mm_P2.50mm -> Capacitor_THT:CP_Radial_D6.3mm_P2.50mm
- J1: footprint (none) -> Connector_RJ:RJ12_Amphenol_54601
- JP1: footprint (none) -> Jumper:SolderJumper-2_P1.3mm_Bridged_RoundedPad1.0x1.5mm
- PTC1: value ~ -> MF-SD013; footprint (none) -> my_lib:ptc-4-mf-sd
- RCPM1, RCPM2, RS1, RTDC1, RTDC2: footprint Resistor_SMD:R_0603_1608Metric_Pad0.98x0.95mm_HandSolder -> Resistor_SMD:R_0603_1608Metric
- RREF1, RV1: footprint Resistor_THT:R_Axial_DIN0309_L9.0mm_D3.2mm_P12.70mm_Horizontal -> Resistor_SMD:R_0603_1608Metric
- RT1, RTAC1, RTAC2, RVP1: footprint Resistor_SMD:R_0201_0603Metric_Pad0.64x0.40mm_HandSolder -> Resistor_SMD:R_0603_1608Metric
- U1: footprint ICS:QFN48_7X7_MCH -> my_lib:QFN50P700X700X90-49N
- U2: footprint ICS:SOIC08_3P9X4P9_BRN -> my_lib:SOIC127P780X210-8N
Connections:
- net VBAT1 is gone; now on net VPP: RVP1.1
- net at C1.1, C5.1, U1.45 (RINGD1)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: now also PTC1.2 (R1)
- net at C3.2, C6.1, U1.46 (TIPD1)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: now also PTC1.4 (R2)
- net at J1.2, RTDC1.1: now also PTC1.1 (R1)
- net at J1.1, RTDC2.1: now also PTC1.3 (R2)
- net 3.3VA renamed +3.3VA
- net VBAT renamed VPP

Commit message: half placed
Parts:
- removed CSWB1: 220uF/25V, Capacitor_THT:CP_Radial_D6.3mm_P2.50mm, symbol Device:C_Polarized_US
- removed J1: 6P2C, Connector_RJ:RJ12_Amphenol_54601, symbol Connector:6P2C
- added J1: 6P2C, Connector_RJ:RJ12_Amphenol_54601, symbol my_lib:6P2C
- C5: footprint Capacitor_SMD:C_0201_0603Metric_Pad0.64x0.40mm_HandSolder -> Capacitor_SMD:C_0603_1608Metric
Connections:
- net +3.3V: no longer CVID1.2, U1.23 (VDDHPI), U1.24 (*ZSI)
- net at PTC1.1 (R1), RTDC1.1: now also J1.4
- net at PTC1.3 (R2), RTDC2.1: now also J1.3
- new net VDDHPI: CVID1.2, U1.23 (VDDHPI), U1.24 (*ZSI)
Changed lines of the file:
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@@
   (junction (at 133.35 120.65) (diameter 0) (color 0 0 0 0)
   )
-  (junction (at 30.48 173.99) (diameter 0) (color 0 0 0 0)
-  )
   (junction (at 260.35 137.16) (diameter 0) (color 0 0 0 0)
   )
@@
   (junction (at 92.71 151.13) (diameter 0) (color 0 0 0 0)
   )
-  (wire (pts (xy 30.48 173.99) (xy 30.48 175.26))
-    (stroke (width 0) (type default))
-  )
   (wire (pts (xy 248.92 148.59) (xy 267.97 148.59))
     (stroke (width 0) (type default))
@@
     (stroke (width 0) (type default))
   )
-  (wire (pts (xy 30.48 186.69) (xy 30.48 182.88))
-    (stroke (width 0) (type default))
-  )
   (wire (pts (xy 55.88 149.86) (xy 55.88 156.21))
     (stroke (width 0) (type default))
@@
     (stroke (width 0) (type default))
   )
-  (wire (pts (xy 30.48 173.99) (xy 24.13 173.99))
-    (stroke (width 0) (type default))
-  )
   (wire (pts (xy 248.92 148.59) (xy 248.92 135.89))
     (stroke (width 0) (type default))
@@
     (stroke (width 0) (type default))
   )
-  (wire (pts (xy 24.13 157.48) (xy 24.13 173.99))
-    (stroke (width 0) (type default))
-  )
   (wire (pts (xy 147.32 96.52) (xy 147.32 101.6))
     (stroke (width 0) (type default))
@@
   )
   (wire (pts (xy 128.27 69.85) (xy 139.7 69.85))
-    (stroke (width 0) (type default))
-  )
-  (wire (pts (xy 30.48 173.99) (xy 39.37 173.99))
     (stroke (width 0) (type default))
   )
@@
   )
   (label "VSW" (at 140.97 163.83 0) (fields_autoplaced)
-    (effects (font (size 1.27 1.27)) (justify left bottom))
-  )
-  (label "VSW" (at 251.46 62.23 0) (fields_autoplaced)
     (effects (font (size 1.27 1.27)) (justify left bottom))
   )
@@
     )
   )
-  (global_label "VDDHPI" (shape passive) (at 39.37 173.99 0) (fields_autoplaced)
-    (effects (font (size 1.27 1.27)) (justify left))
-    (property "Intersheetrefs" "${INTERSHEET_REFS}" (at 47.9984 173.99 0)
-      (effects (font (size 1.27 1.27)) (justify left) hide)
-    )
-  )
   (global_label "INT_N" (shape output) (at 231.14 41.91 0) (fields_autoplaced)
     (effects (font (size 1.27 1.27)) (justify left))
@@
     )
   )
+  (global_label "VSW" (shape passive) (at 254 62.23 0) (fields_autoplaced)
+    (effects (font (size 1.27 1.27)) (justify left))
+    (property "Intersheetrefs" "${INTERSHEET_REFS}" (at 259.544 62.23 0)
+      (effects (font (size 1.27 1.27)) (justify left) hide)
+    )
+  )
   (global_label "FS" (shape input) (at 151.13 54.61 180) (fields_autoplaced)
     (effects (font (size 1.27 1.27)) (justify right))
@@
     (property "Intersheetrefs" "${INTERSHEET_REFS}" (at 155.3604 72.39 0)
       (effects (font (size 1.27 1.27)) (justify right) hide)
-    )
-  )
-  (netclass_flag "" (length 2.54) (shape round) (at 254 62.23 270)
-    (effects (font (size 1.27 1.27)) (justify right bottom))
-    (property "Netclass" "VSW" (at 257.81 62.23 0)
-      (effects (font (size 1.27 1.27) italic) (justify left))
     )
   )
@@
     )
   )
-  (symbol (lib_id "Device:C_Polarized_US") (at 30.48 179.07 0) (unit 1)
-    (in_bom yes) (on_board yes) (dnp no)
-    (property "Reference" "CSWB1" (at 22.86 182.88 0)
-      (effects (font (size 1.27 1.27)) (justify left))
-    )
-    (property "Value" "220uF/25V" (at 31.75 182.88 0)
-      (effects (font (size 1.27 1.27)) (justify left))
-    )
-    (property "Footprint" "Capacitor_THT:CP_Radial_D6.3mm_P2.50mm" (at 30.48 179.07 0)
-      (effects (font (size 1.27 1.27)) hide)
-    )
-    (property "Datasheet" "~" (at 30.48 179.07 0)
-      (effects (font (size 1.27 1.27)) hide)
-    )
-    (pin "1")
-    (pin "2")
-    (instances
-      (project "telluino"
-        (path "/3bd12265-4173-4d6b-91eb-5b474bc7bb16"
-          (reference "CSWB1") (unit 1)
-        )
-        (path "/3bd12265-4173-4d6b-91eb-5b474bc7bb16/de427dad-d24a-4626-86e4-06027dc022b9"
-          (reference "CSWB1") (unit 1)
-        )
-        (path "/3bd12265-4173-4d6b-91eb-5b474bc7bb16/14dbbff9-3cfb-49d8-8c76-2abe81712cc0"
-          (reference "CSWB1") (unit 1)
-        )
-      )
-    )
-  )
   (symbol (lib_id "power:VPP") (at 77.47 88.9 0) (unit 1)
     (in_bom yes) (on_board yes) (dnp no) (fields_autoplaced)
@@
       (effects (font (size 1.27 1.27)))
     )
-    (property "Footprint" "Capacitor_SMD:C_0201_0603Metric_Pad0.64x0.40mm_HandSolder" (at 143.51 77.47 0)
+    (property "Footprint" "Capacitor_SMD:C_0603_1608Metric" (at 143.51 77.47 0)
       (effects (font (size 1.27 1.27)) hide)
     )
@@
     )
   )
-  (symbol (lib_id "power:GNDA") (at 30.48 186.69 0) (unit 1)
-    (in_bom yes) (on_board yes) (dnp no) (fields_autoplaced)
-    (property "Reference" "#PWR013" (at 30.48 193.04 0)
-      (effects (font (size 1.27 1.27)) hide)
-    )
-    (property "Value" "GNDA" (at 30.48 191.77 0)
-      (effects (font (size 1.27 1.27)))
-    )
-    (property "Footprint" "" (at 30.48 186.69 0)
-      (effects (font (size 1.27 1.27)) hide)
-    )
-    (property "Datasheet" "" (at 30.48 186.69 0)
-      (effects (font (size 1.27 1.27)) hide)
-    )
-    (pin "1")
-    (instances
-      (project "telluino"
-        (path "/3bd12265-4173-4d6b-91eb-5b474bc7bb16"
-          (reference "#PWR013") (unit 1)
-        )
-        (path "/3bd12265-4173-4d6b-91eb-5b474bc7bb16/de427dad-d24a-4626-86e4-06027dc022b9"
-          (reference "#PWR010") (unit 1)
-        )
-        (path "/3bd12265-4173-4d6b-91eb-5b474bc7bb16/14dbbff9-3cfb-49d8-8c76-2abe81712cc0"
-          (reference "#PWR021") (unit 1)
-        )
-      )
-    )
-  )
   (symbol (lib_id "power:VPP") (at 143.51 157.48 0) (unit 1)
     (in_bom yes) (on_board yes) (dnp no) (fields_autoplaced)
@@
     )
   )
-  (symbol (lib_id "power:+3.3V") (at 24.13 157.48 0) (unit 1)
-    (in_bom yes) (on_board yes) (dnp no) (fields_autoplaced)
-    (property "Reference" "#PWR021" (at 24.13 161.29 0)
-      (effects (font (size 1.27 1.27)) hide)
-    )
-    (property "Value" "+3.3V" (at 24.13 153.67 0)
-      (effects (font (size 1.27 1.27)))
-    )
-    (property "Footprint" "" (at 24.13 157.48 0)
-      (effects (font (size 1.27 1.27)) hide)
-    )
-    (property "Datasheet" "" (at 24.13 157.48 0)
-      (effects (font (size 1.27 1.27)) hide)
-    )
-    (pin "1")
-    (instances
-      (project "telluino"
-        (path "/3bd12265-4173-4d6b-91eb-5b474bc7bb16/de427dad-d24a-4626-86e4-06027dc022b9"
-          (reference "#PWR021") (unit 1)
-        )
-        (path "/3bd12265-4173-4d6b-91eb-5b474bc7bb16/14dbbff9-3cfb-49d8-8c76-2abe81712cc0"
-          (reference "#PWR010") (unit 1)
-        )
-      )
-    )
-  )
   (symbol (lib_id "Device:R_Small") (at 148.59 59.69 90) (unit 1)
     (in_bom yes) (on_board yes) (dnp no)
@@
     )
   )
-  (symbol (lib_id "Connector:6P2C") (at 30.48 106.68 0) (unit 1)
-    (in_bom yes) (on_board yes) (dnp no) (fields_autoplaced)
-    (property "Reference" "J1" (at 30.48 92.71 0)
-      (effects (font (size 1.27 1.27)))
-    )
-    (property "Value" "6P2C" (at 30.48 95.25 0)
-      (effects (font (size 1.27 1.27)))
-    )
-    (property "Footprint" "Connector_RJ:RJ12_Amphenol_54601" (at 30.48 106.045 90)
-      (effects (font (size 1.27 1.27)) hide)
-    )
-    (property "Datasheet" "~" (at 30.48 106.045 90)
-      (effects (font (size 1.27 1.27)) hide)
-    )
-    (pin "1")
-    (pin "2")
-    (instances
-      (project "telluino"
-        (path "/3bd12265-4173-4d6b-91eb-5b474bc7bb16"
-          (reference "J1") (unit 1)
-        )
-        (path "/3bd12265-4173-4d6b-91eb-5b474bc7bb16/14dbbff9-3cfb-49d8-8c76-2abe81712cc0"
-          (reference "J1") (unit 1)
-        )
-      )
-    )
-  )
   (symbol (lib_id "power:GNDA") (at 134.62 171.45 0) (unit 1)
     (in_bom yes) (on_board yes) (dnp no) (fields_autoplaced)
@@
         )
       )
+    )
+  )
+  (symbol (lib_id "my_lib:6P2C") (at 30.48 106.68 0) (unit 1)
+    (in_bom yes) (on_board yes) (dnp no) (fields_autoplaced)
+    (property "Reference" "J1" (at 30.48 92.71 0)
+      (effects (font (size 1.27 1.27)))
+    )
+    (property "Value" "6P2C" (at 30.48 95.25 0)
+      (effects (font (size 1.27 1.27)))
+    )
+    (property "Footprint" "Connector_RJ:RJ12_Amphenol_54601" (at 30.48 106.045 90)
+      (effects (font (size 1.27 1.27)) hide)
+    )
+    (property "Datasheet" "~" (at 30.48 106.045 90)
+      (effects (font (size 1.27 1.27)) hide)
+    )
+    (pin "1")
+    (pin "2")
+    (pin "3")
+    (pin "4")
+    (pin "5")
+    (pin "6")
+    (instances
+      (project "telluino"
+        (path "/3bd12265-4173-4d6b-91eb-5b474bc7bb16/14dbbff9-3cfb-49d8-8c76-2abe81712cc0"
+          (reference "J1") (unit 1)
+        )
+      )
