File: telluino-kicad/telluino.kicad_pcb (KiCad board)
At the start: 2 copper layers, 92 parts, among them J1 6P2C, J3 USB_B, J4 USB_A, Q2 MMBT3904, Q4 ZXTP2012Z, SW1 SW_Push, U1 LE9641PQC, U10 SS1P3L, U2 TISP61089BDR-S, U3 SS1P3L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

Commit message: half placed
Parts:
- C4: footprint Capacitor_SMD:C_0201_0603Metric_Pad0.64x0.40mm_HandSolder -> Capacitor_SMD:C_0603_1608Metric
- CPF4: value 47uF/100V -> 1uF/100V; footprint Capacitor_THT:CP_Radial_D12.5mm_P5.00mm -> Capacitor_THT:CP_Radial_D8.0mm_P3.50mm
- CSWB1: footprint Capacitor_THT:CP_Radial_D6.3mm_P2.50mm -> Capacitor_THT:CP_Radial_D10.0mm_P5.00mm
- D2: value Red Rx -> RUN Blue
- D3: value Green Tx -> OP Orange
- D5: value RUN Blue -> Green Tx
- D6: value Green Tx -> Red Rx
- D7: value OP Orange -> Green Tx
- moved RVP1 214.5 mm to (77.6, 113.4)
- moved C1 206.8 mm to (77.6, 110.8), turned to 180 degrees
- moved RTAC2 199.7 mm to (95.6, 107.0), turned to 90 degrees
- moved RTDC1 199.1 mm to (92.8, 102.0)
- moved RCPM2 198.0 mm to (90.8, 106.4)
- moved RTDC2 197.4 mm to (92.8, 100.2)
- moved C3 192.3 mm to (90.8, 110.0)
- moved RCPM1 191.8 mm to (99.1, 107.0), turned to 90 degrees
- moved C2 191.1 mm to (90.8, 104.7), turned to 180 degrees
- moved C9 190.4 mm to (96.3, 103.7), turned to 180 degrees
- moved RTAC1 188.2 mm to (97.4, 107.0), turned to 90 degrees
- moved C10 186.6 mm to (95.6, 95.6), turned to 180 degrees
- moved CFL4 184.2 mm to (97.0, 127.6), turned to 90 degrees
- moved RT1 184.2 mm to (97.9, 94.8), turned to -90 degrees
- moved CV2 184.1 mm to (96.3, 98.4)
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Connections:
- CSWB1 pad 1: 3.3V -> +5V
- CVID1 pad 2: 3.3V -> VDDHPI
- D2 pad 1: Net-(D2-K) -> DGND
- D3 pad 1: Net-(D3-K) -> DGND
- D4 pad 1: PD4 -> Net-(D4-K)
- D5 pad 1: DGND -> Net-(D5-K)
- D6 pad 1: PD5 -> PD4
- D7 pad 1: DGND -> PD5
- J1 pad 1: Net-(J1-Pad1) -> unconnected-(J1-Pad1)
- J1 pad 2: Net-(J1-Pad2) -> unconnected-(J1-Pad2)
- J1 pad 3: (no net) -> Net-(J1-Pad3)
- J1 pad 4: (no net) -> Net-(J1-Pad4)
- J1 pad 5: (no net) -> unconnected-(J1-Pad5)
- J1 pad 6: (no net) -> unconnected-(J1-Pad6)
- PTC1 pad 1: Net-(J1-Pad2) -> Net-(J1-Pad4)
- PTC1 pad 3: Net-(J1-Pad1) -> Net-(J1-Pad3)
- RN1 pad 7: Net-(D5-A) -> Net-(D2-A)
- RN1 pad 8: Net-(D7-A) -> Net-(D3-A)
- RN2 pad 1: Net-(D2-A) -> Net-(D4-A)
- RN2 pad 2: Net-(D3-A) -> Net-(D5-A)
- RN2 pad 3: Net-(D6-A) -> Net-(D7-A)
- RN2 pad 4: Net-(D4-A) -> Net-(D6-A)
- RTDC1 pad 1: Net-(J1-Pad1) -> Net-(J1-Pad3)
- RTDC2 pad 1: Net-(J1-Pad2) -> Net-(J1-Pad4)
- U1 pad 23: 3.3V -> VDDHPI
- U1 pad 24: 3.3V -> VDDHPI
- U4 pad 30: Net-(D2-K) -> Net-(D4-K)
- U4 pad 31: Net-(D3-K) -> Net-(D5-K)
- U5 pad 2: Net-(D2-K) -> Net-(D4-K)
- U5 pad 3: Net-(D3-K) -> Net-(D5-K)
