File: telluino-kicad/telluino.kicad_sch (KiCad schematic)
At the start: 26 parts, among them J1 6P2C, U1 LE9641PQC, U2 TISP61089BDR-S

Commit message: before buck supply
Parts:
- added CV1: 4.7uF/8.3V, Capacitor_SMD:C_0201_0603Metric_Pad0.64x0.40mm_HandSolder, symbol Device:C_Small
- added CV2: 1uF/8.3V, Capacitor_SMD:C_0201_0603Metric_Pad0.64x0.40mm_HandSolder, symbol Device:C_Small
- added CVA1: 0.1uF/16V, Capacitor_SMD:C_0201_0603Metric_Pad0.64x0.40mm_HandSolder, symbol Device:C_Small
- added CVD1: 0.01uF/16V, Capacitor_SMD:C_0201_0603Metric_Pad0.64x0.40mm_HandSolder, symbol Device:C_Small
- added CVID1: 0.01uF/18V, Capacitor_SMD:C_0201_0603Metric_Pad0.64x0.40mm_HandSolder, symbol Device:C_Small
- added RV1: 2R0 5%, Resistor_THT:R_Axial_DIN0309_L9.0mm_D3.2mm_P12.70mm_Horizontal, symbol Device:R_Small
- C4: value 0.1 uF/100V -> 0.1 uF/16V; footprint Capacitor_SMD:C_0603_1608Metric_Pad1.08x0.95mm_HandSolder -> Capacitor_SMD:C_0201_0603Metric_Pad0.64x0.40mm_HandSolder
Connections:
- net GNDA: now also C4.1, CV1.1, CV2.1, CVA1.1, CVD1.1, CVID1.1; no longer C4.2
- net at U1.48 (VBAT1): now also C4.2; no longer C4.1
- new net: CV2.2, CVA1.2, RV1.2
- new net: CV1.2, CVD1.2, RV1.1
Other:
- note added: "Locate CVDx near DVDD and CVAx near AVDD pins."
- moved on the sheet: C1, C10, C11, C2, C3, C5, C6, C7, C8, C9, F1, F2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

Commit message: complete_Except_mc
Parts:
- removed C1, C10, C5, C6: 22 nF/100V, Capacitor_SMD:C_0201_0603Metric_Pad0.64x0.40mm_HandSolder, symbol Device:C_Small
- removed C11, C4: 0.1 uF/16V, Capacitor_SMD:C_0201_0603Metric_Pad0.64x0.40mm_HandSolder, symbol Device:C_Small
- removed C2: 0.1 uF/100V, Capacitor_SMD:C_0603_1608Metric_Pad1.08x0.95mm_HandSolder, symbol Device:C_Small
- removed C3: 22 nF/100V, symbol Device:C_Small
- removed C7, C8, C9: 4.7 uF/8.3V, Capacitor_SMD:C_0201_0603Metric_Pad0.64x0.40mm_HandSolder, symbol Device:C_Small
- removed CV1: 4.7uF/8.3V, Capacitor_SMD:C_0201_0603Metric_Pad0.64x0.40mm_HandSolder, symbol Device:C_Small
- removed CV2: 1uF/8.3V, Capacitor_SMD:C_0201_0603Metric_Pad0.64x0.40mm_HandSolder, symbol Device:C_Small
- removed CVA1: 0.1uF/16V, Capacitor_SMD:C_0201_0603Metric_Pad0.64x0.40mm_HandSolder, symbol Device:C_Small
- removed CVD1: 0.01uF/16V, Capacitor_SMD:C_0201_0603Metric_Pad0.64x0.40mm_HandSolder, symbol Device:C_Small
- removed CVID1: 0.01uF/18V, Capacitor_SMD:C_0201_0603Metric_Pad0.64x0.40mm_HandSolder, symbol Device:C_Small
- removed F1: Polyfuse, Resistor_SMD:R_0201_0603Metric, symbol Device:Polyfuse
- removed F2: Polyfuse, symbol Device:Polyfuse
- removed J1: 6P2C, symbol Connector:6P2C
- removed RCPM1, RCPM2, RS1, RTDC1, RTDC2: 1Meg 1%, Resistor_SMD:R_0603_1608Metric_Pad0.98x0.95mm_HandSolder, symbol Device:R
- removed RREF1: 75K 0.5%, Resistor_THT:R_Axial_DIN0309_L9.0mm_D3.2mm_P12.70mm_Horizontal, symbol Device:R_Small
- removed RT1: 47.5K 1%, Resistor_SMD:R_0201_0603Metric_Pad0.64x0.40mm_HandSolder, symbol Device:R_Small
- removed RTAC1, RTAC2: 10K 1%, Resistor_SMD:R_0201_0603Metric_Pad0.64x0.40mm_HandSolder, symbol Device:R_Small
- removed RV1: 2R0 5%, Resistor_THT:R_Axial_DIN0309_L9.0mm_D3.2mm_P12.70mm_Horizontal, symbol Device:R_Small
- removed RVP1: 0, Resistor_SMD:R_0201_0603Metric_Pad0.64x0.40mm_HandSolder, symbol Device:R_Small
- removed U1: LE9641PQC, ICS:QFN48_7X7_MCH, symbol LE9641:LE9641PQC
- removed U2: TISP61089BDR-S, ICS:SOIC08_3P9X4P9_BRN, symbol TISP61089BDR-S:TISP61089BDR-S
Other:
- added sheet arduino_controller (arduino_controllers.kicad_sch)
- added sheet buck_boost_suplly (buck_boot_supply.kicad_sch)
- added sheet connectors (connectors.kicad_sch)
- added sheet slic (slic.kicad_sch)
- note removed: "Locate CVDx near DVDD and CVAx near AVDD pins."
